File: Sidepanel Z- - Kopie/STS1_SIDEPANEL.kicad_sch (KiCad schematic)
At the start: 3 parts, among them J1 Conn_02x04_Odd_Even, J2 Conn_02x02_Odd_Even

Commit message: Review Ready for V2.0
Parts:
- added TP_DEPLOY1, TP_VBAT1: TestPoint, TestPoint:TestPoint_Loop_D1.80mm_Drill1.0mm_Beaded, symbol Connector:TestPoint
- J1: value Conn_02x04_Odd_Even -> (none); footprint SamacSys:M808280842 -> (none)
- J2: value Conn_02x02_Odd_Even -> (none); footprint USER_Passiv:M80-8280442 -> (none)
- Outline1: footprint USER_OUTLINE:OUTLINE_SidepanelY- -> USER_OUTLINE:OUTLINE_SidepanelZ+
Connections:
- new net AntennaDeployment/Deploy: TP_DEPLOY1.1
- new net AntennaDeployment/VBAT: TP_VBAT1.1
Other:
- added sheet AntennaDeployment (AntennaDeployment.kicad_sch)
