File: Sidepanel Z- - Kopie/SolarMPPT.kicad_sch (KiCad schematic)
At the start: 38 parts

Commit message: Review Ready for V2.0
Parts:
- CUR1, CUR2: footprint SOIC127P600X175-8N -> Package_SO:SOIC-8_3.9x4.9mm_P1.27mm
- DOUT1: footprint SamacSys:STMITE -> Diode_SMD:D_0603_1608Metric
- DOUT2: footprint SamacSys:STMITE -> LED_SMD:LED_0603_1608Metric
- L_IN1, L_IN2: footprint SamacSys:INDPM5650X530N -> Inductor_SMD:L_0805_2012Metric
- MPPT1, MPPT2: footprint SamacSys:SOP65P640X120-8N -> Package_SO:TSSOP-8_4.4x3mm_P0.65mm
- SC1, SC2: footprint USER_Activ:3G30A_40x80 -> STS_Connector:3G30A_40x80
Changed lines of the file:
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@@
   )
   (symbol (lib_id "Device:L_Small") (at 100.33 114.3 90) (unit 1)
-    (in_bom yes) (on_board yes) (fields_autoplaced)
+    (in_bom yes) (on_board yes)
     (property "Reference" "L_IN2" (id 0) (at 100.33 109.22 90))
     (property "Value" "10u" (id 1) (at 100.33 111.76 90))
-    (property "Footprint" "SamacSys:INDPM5650X530N" (id 2) (at 100.33 114.3 0)
+    (property "Footprint" "Inductor_SMD:L_0805_2012Metric" (id 2) (at 100.33 114.3 0)
       (effects (font (size 1.27 1.27)) hide)
     )
@@
       (effects (font (size 1.27 1.27)) (justify left))
     )
-    (property "Footprint" "USER_Activ:3G30A_40x80" (id 2) (at 39.37 119.126 90)
+    (property "Footprint" "STS_Connector:3G30A_40x80" (id 2) (at 39.37 119.126 90)
       (effects (font (size 1.27 1.27)) hide)
     )
@@
       (effects (font (size 1.27 1.27)) (justify left))
     )
-    (property "Footprint" "SamacSys:STMITE" (id 2) (at 161.29 97.79 0)
+    (property "Footprint" "LED_SMD:LED_0603_1608Metric" (id 2) (at 161.29 97.79 0)
       (effects (font (size 1.27 1.27)) hide)
     )
@@
     (property "Reference" "MPPT1" (id 0) (at 124.46 39.37 0))
     (property "Value" "SPV1040TTR" (id 1) (at 124.46 41.91 0))
-    (property "Footprint" "SamacSys:SOP65P640X120-8N" (id 2) (at 140.97 44.45 0)
+    (property "Footprint" "Package_SO:TSSOP-8_4.4x3mm_P0.65mm" (id 2) (at 140.97 44.45 0)
       (effects (font (size 1.27 1.27)) (justify left) hide)
     )
@@
       (effects (font (size 1.27 1.27)) (justify right))
     )
-    (property "Footprint" "SOIC127P600X175-8N" (id 2) (at 55.88 74.93 0)
+    (property "Footprint" "Package_SO:SOIC-8_3.9x4.9mm_P1.27mm" (id 2) (at 55.88 74.93 0)
       (effects (font (size 1.27 1.27)) (justify left) hide)
     )
@@
       (effects (font (size 1.27 1.27)) (justify right))
     )
-    (property "Footprint" "SOIC127P600X175-8N" (id 2) (at 55.88 142.24 0)
+    (property "Footprint" "Package_SO:SOIC-8_3.9x4.9mm_P1.27mm" (id 2) (at 55.88 142.24 0)
       (effects (font (size 1.27 1.27)) (justify left) hide)
     )
@@
     (property "Reference" "L_IN1" (id 0) (at 100.33 41.91 90))
     (property "Value" "10u" (id 1) (at 100.33 44.45 90))
-    (property "Footprint" "SamacSys:INDPM5650X530N" (id 2) (at 100.33 46.99 0)
+    (property "Footprint" "Inductor_SMD:L_0805_2012Metric" (id 2) (at 100.33 46.99 0)
       (effects (font (size 1.27 1.27)) hide)
     )
@@
       (effects (font (size 1.27 1.27)) (justify left))
     )
-    (property "Footprint" "SamacSys:STMITE" (id 2) (at 161.29 30.48 0)
+    (property "Footprint" "Diode_SMD:D_0603_1608Metric" (id 2) (at 161.29 30.48 0)
       (effects (font (size 1.27 1.27)) hide)
     )
@@
       (effects (font (size 1.27 1.27)) (justify left))
     )
-    (property "Footprint" "USER_Activ:3G30A_40x80" (id 2) (at 39.37 51.816 90)
+    (property "Footprint" "STS_Connector:3G30A_40x80" (id 2) (at 39.37 51.816 90)
       (effects (font (size 1.27 1.27)) hide)
     )
@@
     (property "Reference" "MPPT2" (id 0) (at 124.46 106.68 0))
     (property "Value" "SPV1040TTR" (id 1) (at 124.46 109.22 0))
-    (property "Footprint" "SamacSys:SOP65P640X120-8N" (id 2) (at 140.97 111.76 0)
-      (effects (font (size 1.27 1.27)) (justify left) hide)
-    )
+    (property "Footprint" "Package_SO:TSSOP-8_4.4x3mm_P0.65mm" (id 2) (at 140.97 111.76 0)
+      (effects (font (size 1.27 1.27)) (justify left) hide)
+    )
