File: Sidepanel Y+/Sensors.kicad_sch (KiCad schematic)
At the start: 8 parts, among them IC1 TMP112AQDRLRQ1, U1 GUVA-C32SM

Commit message: Further fixes, still some open
Connections:
- net VBAT is gone; now on net +3V3: C1.1, U1.4 (VCC)
Changed lines of the file:
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@@
   (junction (at 165.1 46.99) (diameter 0) (color 0 0 0 0)
+  )
+  (junction (at 50.8 34.29) (diameter 0) (color 0 0 0 0)
   )
   (junction (at 50.8 41.91) (diameter 0) (color 0 0 0 0)
@@
     (stroke (width 0) (type default) (color 0 0 0 0))
   )
-  (wire (pts (xy 48.26 46.99) (xy 50.8 46.99))
+  (wire (pts (xy 27.94 46.99) (xy 50.8 46.99))
     (stroke (width 0) (type default) (color 0 0 0 0))
   )
   (wire (pts (xy 165.1 45.72) (xy 165.1 46.99))
+    (stroke (width 0) (type default) (color 0 0 0 0))
+  )
+  (wire (pts (xy 50.8 34.29) (xy 50.8 35.56))
     (stroke (width 0) (type default) (color 0 0 0 0))
   )
@@
     (stroke (width 0) (type default) (color 0 0 0 0))
   )
-  (wire (pts (xy 50.8 33.02) (xy 50.8 35.56))
+  (wire (pts (xy 50.8 33.02) (xy 50.8 34.29))
     (stroke (width 0) (type default) (color 0 0 0 0))
   )
@@
     (stroke (width 0) (type default) (color 0 0 0 0))
   )
+  (wire (pts (xy 27.94 46.99) (xy 27.94 34.29))
+    (stroke (width 0) (type default) (color 0 0 0 0))
+  )
   (wire (pts (xy 165.1 34.29) (xy 165.1 39.37))
     (stroke (width 0) (type default) (color 0 0 0 0))
@@
     (stroke (width 0) (type default) (color 0 0 0 0))
   )
-  (hierarchical_label "VBAT" (shape input) (at 48.26 46.99 180)
-    (effects (font (size 1.27 1.27)) (justify right))
-  )
-  (hierarchical_label "VBAT" (shape input) (at 48.26 46.99 180)
-    (effects (font (size 1.27 1.27)) (justify right))
+  (wire (pts (xy 27.94 34.29) (xy 50.8 34.29))
+    (stroke (width 0) (type default) (color 0 0 0 0))
   )
   (hierarchical_label "SDA_TMP" (shape bidirectional) (at 166.37 46.99 0)
