File: Sidepanel Y+/STS1_SIDEPANEL.kicad_sch (KiCad schematic)
At the start: 4 parts, among them J1 ZF5S-08-01-T-WT

Commit message: small adjustments
Parts:
- removed J1: ZF5S-08-01-T-WT, STS_connector:SAMTEC_ZF5S-08-01-T-WT, symbol EPS connector:ZF5S-08-01-T-WT
- added J1: Conn_01x08, STS_connector:SAMTEC_ZF5S-08-01-T-WT, symbol Connector_Generic:Conn_01x08
Connections:
- net GND: now also J1.05 (Pin_5)
- net MPPT1: now also J1.06 (Pin_6)
- net MPPT2: now also J1.03 (Pin_3)
- net SC1_I+: now also J1.07 (Pin_7)
- net SC1_V+: now also J1.08 (Pin_8)
- net SC2_I+: now also J1.02 (Pin_2)
- net SC2_V+: now also J1.01 (Pin_1)
- net TEMP+: now also J1.04 (Pin_4)
- no-connect marks 0 -> 2

Commit message: added the libraries for the specific components
Parts:
- J1: footprint STS_connector:SAMTEC_ZF5S-08-01-T-WT -> STS_Connector:SAMTEC_ZF5S-08-01-T-WT
- UV1: footprint STS_connector:5014610491 -> STS_Connector:5014610491
Changed lines of the file:
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@@
       (effects (font (size 1.27 1.27)) hide)
     )
-    (property "Footprint" "STS_connector:5014610491" (id 2) (at 95.504 76.454 0)
+    (property "Footprint" "STS_Connector:5014610491" (id 2) (at 95.504 76.454 0)
       (effects (font (size 1.27 1.27)) hide)
     )
@@
     (property "Reference" "J1" (id 0) (at 65.024 64.516 0))
     (property "Value" "Conn_01x08" (id 1) (at 65.024 67.056 0))
-    (property "Footprint" "STS_connector:SAMTEC_ZF5S-08-01-T-WT" (id 2) (at 65.024 81.026 0)
+    (property "Footprint" "STS_Connector:SAMTEC_ZF5S-08-01-T-WT" (id 2) (at 65.024 81.026 0)
       (effects (font (size 1.27 1.27)) hide)
     )
@@
     )
     (path "/9800fec4-2f70-44cf-84e6-22af43c255e5"
-      (reference "J1") (unit 1) (value "Conn_01x08") (footprint "STS_connector:SAMTEC_ZF5S-08-01-T-WT")
+      (reference "J1") (unit 1) (value "Conn_01x08") (footprint "STS_Connector:SAMTEC_ZF5S-08-01-T-WT")
     )
     (path "/4f87559b-6bba-4ff6-97a7-dad9a308db2d/bfe4e68f-4cef-4b31-adff-8df094bc3870"
@@
     )
     (path "/4f87559b-6bba-4ff6-97a7-dad9a308db2d/e7b54c2f-482e-4a97-841f-62a80e0193a8"
-      (reference "SC1") (unit 1) (value "Solar_Cell") (footprint "STS_Solarcells:3G30A_40x80")
+      (reference "SC1") (unit 1) (value "Solar_Cell") (footprint "STS_solder:3G30A_40x80_Y_SC1")
     )
     (path "/4f87559b-6bba-4ff6-97a7-dad9a308db2d/3ad17c33-30d5-4097-824f-a9c26e6ca325"
-      (reference "SC2") (unit 1) (value "Solar_Cell") (footprint "STS_Solarcells:3G30A_40x80")
+      (reference "SC2") (unit 1) (value "Solar_Cell") (footprint "STS_solder:3G30A_40x80_Y_SC2")
     )
     (path "/cd74d053-e62a-45a3-9f24-631862f85655"
@@
     )
     (path "/51a1d03d-d1b0-433b-a1de-be96d363771f"
-      (reference "UV1") (unit 1) (value "501461-0491") (footprint "STS_connector:5014610491")
-    )
-  )
+      (reference "UV1") (unit 1) (value "501461-0491") (footprint "STS_Connector:5014610491")
+    )
+  )
