File: Muster/STS1_SIDEPANEL.kicad_pcb (KiCad board)
At the start: 2 copper layers, 98 x 98 mm, 56 parts, among them IC1 TMP112AQDRLRQ1, J1 Conn_02x04_Odd_Even, J2 Conn_02x02_Odd_Even, Q1 BSS214NW, U1 GUVA-C32SM

Commit message: changed the outline of the pcbs + new axis orientaion + changed the footprint of the solar cells
Parts:
- added D1: PMEG2020EH, Diode_SMD:D_SOD-123F, B.Cu at (112.3, 67.9)
- added D2: PMEG2020EH, Diode_SMD:D_SOD-123F, B.Cu at (140.2, 109.7)
Routing:
- net /SolarMPPT/MPPT2_OUT: track 14.5 -> 26.5 mm
- net /SolarMPPT/MPPT2_IN: track 6.57 -> 15.4 mm
- net /SolarMPPT/MPPT1_IN: track 6.57 -> 15.3 mm
- net /SolarMPPT/MPPT1_OUT: track 14.5 -> 22.4 mm
- net GND: vias 296 -> 293
