File: Muster/SolarMPPT.kicad_sch (KiCad schematic)
At the start: 38 parts

Commit message: changed the outline of the pcbs + new axis orientaion + changed the footprint of the solar cells
Parts:
- added D1, D2: PMEG2020EH, Diode_SMD:D_SOD-123F, symbol Diode:PMEG2020EH
Connections:
- net MPPT1_IN: now also D1.2 (A)
- net MPPT1_OUT: now also D1.1 (K)
- net MPPT2_IN: now also D2.2 (A)
- net MPPT2_OUT: now also D2.1 (K)
Changed lines of the file:
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@@
   (junction (at 153.67 46.99) (diameter 0) (color 0 0 0 0)
   )
+  (junction (at 146.05 43.18) (diameter 0) (color 0 0 0 0)
+  )
   (junction (at 58.42 81.28) (diameter 0) (color 0 0 0 0)
   )
@@
   (junction (at 148.59 57.15) (diameter 0) (color 0 0 0 0)
   )
+  (junction (at 146.05 110.49) (diameter 0) (color 0 0 0 0)
+  )
   (junction (at 58.42 46.99) (diameter 0) (color 0 0 0 0)
   )
@@
   (junction (at 153.67 114.3) (diameter 0) (color 0 0 0 0)
   )
+  (junction (at 104.14 101.6) (diameter 0) (color 0 0 0 0)
+  )
   (junction (at 153.67 121.92) (diameter 0) (color 0 0 0 0)
   )
@@
   (junction (at 81.28 114.3) (diameter 0) (color 0 0 0 0)
   )
+  (junction (at 104.14 35.56) (diameter 0) (color 0 0 0 0)
+  )
   (junction (at 81.28 46.99) (diameter 0) (color 0 0 0 0)
   )
@@
     (stroke (width 0) (type default) (color 0 0 0 0))
   )
-  (wire (pts (xy 104.14 39.37) (xy 104.14 46.99))
+  (wire (pts (xy 104.14 35.56) (xy 104.14 46.99))
     (stroke (width 0) (type default) (color 0 0 0 0))
   )
@@
     (stroke (width 0) (type default) (color 0 0 0 0))
   )
+  (wire (pts (xy 127 101.6) (xy 146.05 101.6))
+    (stroke (width 0) (type default) (color 0 0 0 0))
+  )
   (wire (pts (xy 149.86 54.61) (xy 153.67 54.61))
     (stroke (width 0) (type default) (color 0 0 0 0))
@@
     (stroke (width 0) (type default) (color 0 0 0 0))
   )
+  (wire (pts (xy 146.05 35.56) (xy 146.05 43.18))
+    (stroke (width 0) (type default) (color 0 0 0 0))
+  )
   (wire (pts (xy 81.28 116.84) (xy 81.28 114.3))
     (stroke (width 0) (type default) (color 0 0 0 0))
@@
     (stroke (width 0) (type default) (color 0 0 0 0))
   )
+  (wire (pts (xy 129.54 35.56) (xy 146.05 35.56))
+    (stroke (width 0) (type default) (color 0 0 0 0))
+  )
   (wire (pts (xy 166.37 43.18) (xy 167.64 43.18))
     (stroke (width 0) (type default) (color 0 0 0 0))
@@
     (stroke (width 0) (type default) (color 0 0 0 0))
   )
+  (wire (pts (xy 121.92 35.56) (xy 104.14 35.56))
+    (stroke (width 0) (type default) (color 0 0 0 0))
+  )
   (wire (pts (xy 154.94 95.25) (xy 154.94 90.17))
     (stroke (width 0) (type default) (color 0 0 0 0))
@@
     (stroke (width 0) (type default) (color 0 0 0 0))
   )
+  (wire (pts (xy 104.14 101.6) (xy 119.38 101.6))
+    (stroke (width 0) (type default) (color 0 0 0 0))
+  )
   (wire (pts (xy 58.42 146.05) (xy 58.42 148.59))
     (stroke (width 0) (type default) (color 0 0 0 0))
@@
     (stroke (width 0) (type default) (color 0 0 0 0))
   )
+  (wire (pts (xy 104.14 101.6) (xy 104.14 114.3))
+    (stroke (width 0) (type default) (color 0 0 0 0))
+  )
   (wire (pts (xy 66.04 78.74) (xy 66.04 80.01))
     (stroke (width 0) (type default) (color 0 0 0 0))
@@
     (stroke (width 0) (type default) (color 0 0 0 0))
   )
-  (wire (pts (xy 104.14 105.41) (xy 104.14 114.3))
+  (wire (pts (xy 104.14 95.25) (xy 104.14 101.6))
     (stroke (width 0) (type default) (color 0 0 0 0))
   )
@@
     (stroke (width 0) (type default) (color 0 0 0 0))
   )
+  (wire (pts (xy 146.05 101.6) (xy 146.05 110.49))
+    (stroke (width 0) (type default) (color 0 0 0 0))
+  )
   (wire (pts (xy 176.53 119.38) (xy 176.53 124.46))
     (stroke (width 0) (type default) (color 0 0 0 0))
@@
   )
   (wire (pts (xy 144.78 114.3) (xy 146.05 114.3))
+    (stroke (width 0) (type default) (color 0 0 0 0))
+  )
+  (wire (pts (xy 104.14 29.21) (xy 104.14 35.56))
     (stroke (width 0) (type default) (color 0 0 0 0))
   )
@@
     )
     (pin "1")
+  )
+  (symbol (lib_id "Diode:PMEG2020EH") (at 123.19 101.6 0) (mirror y) (unit 1)
+    (in_bom yes) (on_board yes) (fields_autoplaced)
+    (property "Reference" "D2" (id 0) (at 123.5075 95.25 0))
+    (property "Value" "PMEG2020EH" (id 1) (at 123.5075 97.79 0))
+    (property "Footprint" "Diode_SMD:D_SOD-123F" (id 2) (at 123.19 106.045 0)
+      (effects (font (size 1.27 1.27)) hide)
+    )
+    (property "Datasheet" "https://assets.nexperia.com/documents/data-sheet/PMEG2020EH_EJ.pdf" (id 3) (at 123.19 101.6 0)
+      (effects (font (size 1.27 1.27)) hide)
+    )
+    (pin "1")
+    (pin "2")
   )
   (symbol (lib_id "power:GND") (at 66.04 80.01 0) (unit 1)
@@
     (pin "1")
   )
+  (symbol (lib_id "Diode:PMEG2020EH") (at 125.73 35.56 0) (mirror y) (unit 1)
+    (in_bom yes) (on_board yes) (fields_autoplaced)
+    (property "Reference" "D1" (id 0) (at 126.0475 29.21 0))
+    (property "Value" "PMEG2020EH" (id 1) (at 126.0475 31.75 0))
+    (property "Footprint" "Diode_SMD:D_SOD-123F" (id 2) (at 125.73 40.005 0)
+      (effects (font (size 1.27 1.27)) hide)
+    )
+    (property "Datasheet" "https://assets.nexperia.com/documents/data-sheet/PMEG2020EH_EJ.pdf" (id 3) (at 125.73 35.56 0)
+      (effects (font (size 1.27 1.27)) hide)
+    )
+    (pin "1")
+    (pin "2")
+  )
   (symbol (lib_id "SamacSys:SPV1040TTR") (at 104.14 114.3 0) (unit 1)
