File: Sidepanel X+/SolarMPPT.kicad_sch (KiCad schematic)
At the start: 19 parts

Commit message: Review Ready for V2.0
Parts:
- CUR1: footprint SOIC127P600X175-8N -> Package_SO:SOIC-8_3.9x4.9mm_P1.27mm
- DOUT1: footprint SamacSys:STMITE -> Diode_SMD:D_0603_1608Metric
- L_IN1: footprint SamacSys:INDPM5650X530N -> Inductor_SMD:L_0805_2012Metric
- MPPT1: footprint SamacSys:SOP65P640X120-8N -> Package_SO:TSSOP-8_4.4x3mm_P0.65mm
- SC1: footprint USER_Activ:3G30A_40x80 -> STS_Connector:3G30A_40x80
Changed lines of the file:
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@@
     (property "Reference" "MPPT1" (id 0) (at 124.46 39.37 0))
     (property "Value" "SPV1040TTR" (id 1) (at 124.46 41.91 0))
-    (property "Footprint" "SamacSys:SOP65P640X120-8N" (id 2) (at 140.97 44.45 0)
+    (property "Footprint" "Package_SO:TSSOP-8_4.4x3mm_P0.65mm" (id 2) (at 140.97 44.45 0)
       (effects (font (size 1.27 1.27)) (justify left) hide)
     )
@@
       (effects (font (size 1.27 1.27)) (justify right))
     )
-    (property "Footprint" "SOIC127P600X175-8N" (id 2) (at 55.88 74.93 0)
+    (property "Footprint" "Package_SO:SOIC-8_3.9x4.9mm_P1.27mm" (id 2) (at 55.88 74.93 0)
       (effects (font (size 1.27 1.27)) (justify left) hide)
     )
@@
     (property "Reference" "L_IN1" (id 0) (at 100.33 41.91 90))
     (property "Value" "10u" (id 1) (at 100.33 44.45 90))
-    (property "Footprint" "SamacSys:INDPM5650X530N" (id 2) (at 100.33 46.99 0)
+    (property "Footprint" "Inductor_SMD:L_0805_2012Metric" (id 2) (at 100.33 46.99 0)
       (effects (font (size 1.27 1.27)) hide)
     )
@@
       (effects (font (size 1.27 1.27)) (justify left))
     )
-    (property "Footprint" "SamacSys:STMITE" (id 2) (at 161.29 30.48 0)
+    (property "Footprint" "Diode_SMD:D_0603_1608Metric" (id 2) (at 161.29 30.48 0)
       (effects (font (size 1.27 1.27)) hide)
     )
@@
       (effects (font (size 1.27 1.27)) (justify left))
     )
-    (property "Footprint" "USER_Activ:3G30A_40x80" (id 2) (at 39.37 51.816 90)
-      (effects (font (size 1.27 1.27)) hide)
-    )
+    (property "Footprint" "STS_Connector:3G30A_40x80" (id 2) (at 39.37 51.816 90)
+      (effects (font (size 1.27 1.27)) hide)
+    )

Commit message: Next fix
Parts:
- SC1: value Solar_Cell -> (none); footprint STS_Connector:3G30A_40x80 -> (none)
Changed lines of the file:
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@@
       (effects (font (size 1.27 1.27)) (justify left))
     )
-    (property "Value" "Solar_Cell" (id 1) (at 43.18 52.4509 0)
+    (property "Value" "" (id 1) (at 43.18 52.4509 0)
       (effects (font (size 1.27 1.27)) (justify left))
     )
-    (property "Footprint" "STS_Connector:3G30A_40x80" (id 2) (at 39.37 51.816 90)
+    (property "Footprint" "" (id 2) (at 39.37 51.816 90)
       (effects (font (size 1.27 1.27)) hide)
     )

Commit message: release_2.0, Ordered PCBs
Parts:
- DOUT1: footprint Diode_SMD:D_0603_1608Metric -> SamacSys:STMITE
- L_IN1: value 10u -> (none); footprint Inductor_SMD:L_0805_2012Metric -> (none)
- SC1: value (none) -> Solar_Cell; footprint (none) -> STS_Solarcells:3G30A_40x80
Changed lines of the file:
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@@
     (in_bom yes) (on_board yes) (fields_autoplaced)
     (property "Reference" "L_IN1" (id 0) (at 100.33 41.91 90))
-    (property "Value" "10u" (id 1) (at 100.33 44.45 90))
-    (property "Footprint" "Inductor_SMD:L_0805_2012Metric" (id 2) (at 100.33 46.99 0)
+    (property "Value" "" (id 1) (at 100.33 44.45 90))
+    (property "Footprint" "" (id 2) (at 100.33 46.99 0)
       (effects (font (size 1.27 1.27)) hide)
     )
@@
       (effects (font (size 1.27 1.27)) (justify left))
     )
-    (property "Footprint" "Diode_SMD:D_0603_1608Metric" (id 2) (at 161.29 30.48 0)
+    (property "Footprint" "SamacSys:STMITE" (id 2) (at 161.29 30.48 0)
       (effects (font (size 1.27 1.27)) hide)
     )
@@
       (effects (font (size 1.27 1.27)) (justify left))
     )
-    (property "Value" "" (id 1) (at 43.18 52.4509 0)
+    (property "Value" "Solar_Cell" (id 1) (at 43.18 52.4509 0)
       (effects (font (size 1.27 1.27)) (justify left))
     )
-    (property "Footprint" "" (id 2) (at 39.37 51.816 90)
+    (property "Footprint" "STS_Solarcells:3G30A_40x80" (id 2) (at 39.37 51.816 90)
       (effects (font (size 1.27 1.27)) hide)
     )

Commit message: Diode D1 angebracht
Parts:
- added D1: PMEG2020EH, Diode_SMD:D_SOD-123F, symbol Diode:PMEG2020EH
- L_IN1: value (none) -> 10u; footprint (none) -> STS_Inductor_SMD:XAL6060103MEC
Connections:
- net MPPT1_IN: now also D1.2 (A)
- net MPPT1_OUT: now also D1.1 (K)
Changed lines of the file:
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@@
   (junction (at 153.67 46.99) (diameter 0) (color 0 0 0 0)
   )
+  (junction (at 104.14 33.02) (diameter 0) (color 0 0 0 0)
+  )
   (junction (at 58.42 81.28) (diameter 0) (color 0 0 0 0)
   )
@@
   (junction (at 39.37 46.99) (diameter 0) (color 0 0 0 0)
   )
+  (junction (at 146.05 43.18) (diameter 0) (color 0 0 0 0)
+  )
   (junction (at 95.25 46.99) (diameter 0) (color 0 0 0 0)
   )
@@
     (stroke (width 0) (type default) (color 0 0 0 0))
   )
-  (wire (pts (xy 104.14 39.37) (xy 104.14 46.99))
+  (wire (pts (xy 104.14 27.94) (xy 104.14 33.02))
+    (stroke (width 0) (type default) (color 0 0 0 0))
+  )
+  (wire (pts (xy 146.05 33.02) (xy 146.05 43.18))
     (stroke (width 0) (type default) (color 0 0 0 0))
   )
@@
     (stroke (width 0) (type default) (color 0 0 0 0))
   )
+  (wire (pts (xy 104.14 33.02) (xy 104.14 46.99))
+    (stroke (width 0) (type default) (color 0 0 0 0))
+  )
   (wire (pts (xy 190.5 57.15) (xy 190.5 64.77))
     (stroke (width 0) (type default) (color 0 0 0 0))
@@
     (stroke (width 0) (type default) (color 0 0 0 0))
   )
+  (wire (pts (xy 104.14 33.02) (xy 120.65 33.02))
+    (stroke (width 0) (type default) (color 0 0 0 0))
+  )
   (wire (pts (xy 166.37 46.99) (xy 165.1 46.99))
+    (stroke (width 0) (type default) (color 0 0 0 0))
+  )
+  (wire (pts (xy 128.27 33.02) (xy 146.05 33.02))
     (stroke (width 0) (type default) (color 0 0 0 0))
   )
@@
     (in_bom yes) (on_board yes) (fields_autoplaced)
     (property "Reference" "L_IN1" (id 0) (at 100.33 41.91 90))
-    (property "Value" "" (id 1) (at 100.33 44.45 90))
-    (property "Footprint" "" (id 2) (at 100.33 46.99 0)
+    (property "Value" "10u" (id 1) (at 100.33 44.45 90))
+    (property "Footprint" "STS_Inductor_SMD:XAL6060103MEC" (id 2) (at 100.33 46.99 0)
       (effects (font (size 1.27 1.27)) hide)
     )
@@
       (effects (font (size 1.27 1.27)) hide)
     )
+    (pin "1")
+    (pin "2")
+  )
+  (symbol (lib_id "Diode:PMEG2020EH") (at 124.46 33.02 0) (mirror y) (unit 1)
+    (in_bom yes) (on_board yes) (fields_autoplaced)
+    (property "Reference" "D1" (id 0) (at 124.7775 26.67 0))
+    (property "Value" "PMEG2020EH" (id 1) (at 124.7775 29.21 0))
+    (property "Footprint" "Diode_SMD:D_SOD-123F" (id 2) (at 124.46 37.465 0)
+      (effects (font (size 1.27 1.27)) hide)
+    )
+    (property "Datasheet" "https://assets.nexperia.com/documents/data-sheet/PMEG2020EH_EJ.pdf" (id 3) (at 124.46 33.02 0)
+      (effects (font (size 1.27 1.27)) hide)
+    )

Commit message: changes to the solar cells footprint, added camera mounts
Parts:
- L_IN1: footprint STS_Inductor_SMD:XAL6060103MEC -> STS_Inductor_SMD:IND_XAL6060-103MEC
Changed lines of the file:
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@@
     (property "Reference" "L_IN1" (id 0) (at 100.33 41.91 90))
     (property "Value" "10u" (id 1) (at 100.33 44.45 90))
-    (property "Footprint" "STS_Inductor_SMD:XAL6060103MEC" (id 2) (at 100.33 46.99 0)
+    (property "Footprint" "STS_Inductor_SMD:IND_XAL6060-103MEC" (id 2) (at 100.33 46.99 0)
       (effects (font (size 1.27 1.27)) hide)
     )

Commit message: small adjustments
Parts:
- L_IN1: footprint STS_Inductor_SMD:IND_XAL6060-103MEC -> STS_Inductor_SMD:XAL6060103MEC
- R21: value tbd -> 330k
Changed lines of the file:
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@@
   (junction (at 153.67 46.99) (diameter 0) (color 0 0 0 0)
   )
-  (junction (at 104.14 33.02) (diameter 0) (color 0 0 0 0)
-  )
   (junction (at 58.42 81.28) (diameter 0) (color 0 0 0 0)
   )
@@
   (junction (at 148.59 57.15) (diameter 0) (color 0 0 0 0)
   )
+  (junction (at 144.78 46.99) (diameter 0) (color 0 0 0 0)
+  )
   (junction (at 58.42 46.99) (diameter 0) (color 0 0 0 0)
   )
@@
   (junction (at 39.37 46.99) (diameter 0) (color 0 0 0 0)
   )
-  (junction (at 146.05 43.18) (diameter 0) (color 0 0 0 0)
-  )
   (junction (at 95.25 46.99) (diameter 0) (color 0 0 0 0)
   )
@@
   (junction (at 81.28 46.99) (diameter 0) (color 0 0 0 0)
   )
+  (junction (at 104.14 31.75) (diameter 0) (color 0 0 0 0)
+  )
   (junction (at 95.25 54.61) (diameter 0) (color 0 0 0 0)
   )
@@
     (stroke (width 0) (type default) (color 0 0 0 0))
   )
-  (wire (pts (xy 104.14 27.94) (xy 104.14 33.02))
-    (stroke (width 0) (type default) (color 0 0 0 0))
-  )
-  (wire (pts (xy 146.05 33.02) (xy 146.05 43.18))
-    (stroke (width 0) (type default) (color 0 0 0 0))
-  )
   (wire (pts (xy 148.59 57.15) (xy 148.59 54.61))
     (stroke (width 0) (type default) (color 0 0 0 0))
@@
     (stroke (width 0) (type default) (color 0 0 0 0))
   )
+  (wire (pts (xy 104.14 31.75) (xy 120.65 31.75))
+    (stroke (width 0) (type default) (color 0 0 0 0))
+  )
   (wire (pts (xy 144.78 52.07) (xy 149.86 52.07))
     (stroke (width 0) (type default) (color 0 0 0 0))
@@
     (stroke (width 0) (type default) (color 0 0 0 0))
   )
+  (wire (pts (xy 104.14 26.67) (xy 104.14 31.75))
+    (stroke (width 0) (type default) (color 0 0 0 0))
+  )
   (wire (pts (xy 60.96 46.99) (xy 60.96 48.26))
     (stroke (width 0) (type default) (color 0 0 0 0))
@@
     (stroke (width 0) (type default) (color 0 0 0 0))
   )
-  (wire (pts (xy 104.14 33.02) (xy 104.14 46.99))
-    (stroke (width 0) (type default) (color 0 0 0 0))
-  )
   (wire (pts (xy 190.5 57.15) (xy 190.5 64.77))
     (stroke (width 0) (type default) (color 0 0 0 0))
@@
     (stroke (width 0) (type default) (color 0 0 0 0))
   )
+  (wire (pts (xy 100.33 52.07) (xy 104.14 52.07))
+    (stroke (width 0) (type default) (color 0 0 0 0))
+  )
   (wire (pts (xy 190.5 43.18) (xy 176.53 43.18))
     (stroke (width 0) (type default) (color 0 0 0 0))
@@
     (stroke (width 0) (type default) (color 0 0 0 0))
   )
-  (wire (pts (xy 104.14 52.07) (xy 100.33 52.07))
-    (stroke (width 0) (type default) (color 0 0 0 0))
-  )
   (wire (pts (xy 66.04 46.99) (xy 66.04 48.26))
     (stroke (width 0) (type default) (color 0 0 0 0))
@@
     (stroke (width 0) (type default) (color 0 0 0 0))
   )
+  (wire (pts (xy 144.78 31.75) (xy 144.78 46.99))
+    (stroke (width 0) (type default) (color 0 0 0 0))
+  )
   (wire (pts (xy 176.53 57.15) (xy 148.59 57.15))
     (stroke (width 0) (type default) (color 0 0 0 0))
@@
     (stroke (width 0) (type default) (color 0 0 0 0))
   )
+  (wire (pts (xy 104.14 31.75) (xy 104.14 46.99))
+    (stroke (width 0) (type default) (color 0 0 0 0))
+  )
   (wire (pts (xy 148.59 64.77) (xy 148.59 63.5))
     (stroke (width 0) (type default) (color 0 0 0 0))
@@
     (stroke (width 0) (type default) (color 0 0 0 0))
   )
-  (wire (pts (xy 104.14 33.02) (xy 120.65 33.02))
+  (wire (pts (xy 128.27 31.75) (xy 144.78 31.75))
     (stroke (width 0) (type default) (color 0 0 0 0))
   )
   (wire (pts (xy 166.37 46.99) (xy 165.1 46.99))
-    (stroke (width 0) (type default) (color 0 0 0 0))
-  )
-  (wire (pts (xy 128.27 33.02) (xy 146.05 33.02))
     (stroke (width 0) (type default) (color 0 0 0 0))
   )
@@
   (hierarchical_label "MPPT1" (shape output) (at 195.58 43.18 0)
     (effects (font (size 1.27 1.27)) (justify left))
+  )
+  (symbol (lib_id "Diode:PMEG2020EH") (at 124.46 31.75 0) (mirror y) (unit 1)
+    (in_bom yes) (on_board yes) (fields_autoplaced)
+    (property "Reference" "D1" (id 0) (at 124.7775 25.4 0))
+    (property "Value" "PMEG2020EH" (id 1) (at 124.7775 27.94 0))
+    (property "Footprint" "Diode_SMD:D_SOD-123F" (id 2) (at 124.46 36.195 0)
+      (effects (font (size 1.27 1.27)) hide)
+    )
+    (property "Datasheet" "https://assets.nexperia.com/documents/data-sheet/PMEG2020EH_EJ.pdf" (id 3) (at 124.46 31.75 0)
+      (effects (font (size 1.27 1.27)) hide)
+    )
+    (pin "1")
+    (pin "2")
   )
   (symbol (lib_id "Device:R_Small") (at 170.18 43.18 270) (unit 1)
@@
       (effects (font (size 1.27 1.27)) (justify right))
     )
-    (property "Value" "tbd" (id 1) (at 179.07 62.2299 0)
+    (property "Value" "330k" (id 1) (at 179.07 62.2299 0)
       (effects (font (size 1.27 1.27)) (justify right))
     )
@@
     (property "Reference" "L_IN1" (id 0) (at 100.33 41.91 90))
     (property "Value" "10u" (id 1) (at 100.33 44.45 90))
-    (property "Footprint" "STS_Inductor_SMD:IND_XAL6060-103MEC" (id 2) (at 100.33 46.99 0)
+    (property "Footprint" "STS_Inductor_SMD:XAL6060103MEC" (id 2) (at 100.33 46.99 0)
       (effects (font (size 1.27 1.27)) hide)
     )
@@
       (effects (font (size 1.27 1.27)) hide)
     )
-    (pin "1")
-    (pin "2")
-  )
-  (symbol (lib_id "Diode:PMEG2020EH") (at 124.46 33.02 0) (mirror y) (unit 1)
-    (in_bom yes) (on_board yes) (fields_autoplaced)
-    (property "Reference" "D1" (id 0) (at 124.7775 26.67 0))
-    (property "Value" "PMEG2020EH" (id 1) (at 124.7775 29.21 0))
-    (property "Footprint" "Diode_SMD:D_SOD-123F" (id 2) (at 124.46 37.465 0)
-      (effects (font (size 1.27 1.27)) hide)
-    )
-    (property "Datasheet" "https://assets.nexperia.com/documents/data-sheet/PMEG2020EH_EJ.pdf" (id 3) (at 124.46 33.02 0)
-      (effects (font (size 1.27 1.27)) hide)
-    )

Commit message: small adjustments
Parts:
- SC1: footprint STS_Solarcells:3G30A_40x80 -> STS_solder:3G30A_40x80
Changed lines of the file:
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@@
       (effects (font (size 1.27 1.27)) (justify left))
     )
-    (property "Footprint" "STS_Solarcells:3G30A_40x80" (id 2) (at 39.37 51.816 90)
+    (property "Footprint" "STS_solder:3G30A_40x80" (id 2) (at 39.37 51.816 90)
       (effects (font (size 1.27 1.27)) hide)
     )
