File: Flex_PCBs/SP_to_EDU/SP_EDU_Cam_Z_Flex/SP_EDU_Cam_Z_Flex.kicad_pcb (KiCad board)
At the start: 2 copper layers, 11.4 x 64 mm, 2 parts, among them J1 Conn_01x22_Male, J2 Conn_01x22_Male

Commit message: Update SP_EDU_Z_Flex for FM
Other:
- board text added: "SP_EDU_Cam_Z_Flex_V1.0"
- board text removed: "SP_EDU_Cam_ZM_Flex_V1.0"
Changed lines of the file:
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@@
 		(layer "User.1")
 	)
-	(gr_text "SP_EDU_Cam_ZM_Flex_V1.0"
-		(at 135.05 96.9 -90)
+	(gr_text "SP_EDU_Cam_Z_Flex_V1.0"
+		(at 132.35 128 90)
 		(layer "F.SilkS")
 		(effects
