File: Sidepanel Y/STS1_SIDEPANEL.kicad_pcb (KiCad board)
At the start: 4 copper layers, 82.8 x 100 mm, 47 parts, among them IC1 TMP112AQDRLRQ1, J1 Conn_01x08, U1 GUVA-C32SM, U11 INA180A4, U12 INA180A4

Commit message: generated the gerber files for ordering
Parts:
- added ?: , , F.Cu at (130.8, 90.9)
- added ?: , , F.Cu at (124.1, 85.7)
Changed lines of the file:
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@@
 		)
 	)
+	(footprint ""
+		(layer "F.Cu")
+		(at 130.8 90.93)
+		(property "Reference" ""
+			(at 0 0 0)
+			(layer "F.SilkS")
+			(effects
+				(font
+					(size 1.27 1.27)
+					(thickness 0.15)
+				)
+			)
+		)
+		(property "Value" ""
+			(at 0 0 0)
+			(layer "F.Fab")
+			(effects
+				(font
+					(size 1.27 1.27)
+					(thickness 0.15)
+				)
+			)
+		)
+		(property "Footprint" ""
+			(at 0 0 0)
+			(layer "F.Fab")
+			(hide yes)
+			(effects
+				(font
+					(size 1.27 1.27)
+					(thickness 0.15)
+				)
+			)
+		)
+		(property "Datasheet" ""
+			(at 0 0 0)
+			(layer "F.Fab")
+			(hide yes)
+			(effects
+				(font
+					(size 1.27 1.27)
+					(thickness 0.15)
+				)
+			)
+		)
+		(property "Description" ""
+			(at 0 0 0)
+			(layer "F.Fab")
+			(hide yes)
+			(effects
+				(font
+					(size 1.27 1.27)
+					(thickness 0.15)
+				)
+			)
+		)
+		(pad "" smd roundrect
+			(at -0.0205 0 180)
+			(size 0.9 0.95)
+			(layers "B.Cu" "B.Paste" "B.Mask")
+			(roundrect_rratio 0.25)
+			(net 1 "GND")
+			(pintype "passive")
+		)
+	)
 	(footprint "STS_solder:3G30A_40x80_Y_SC1"
 		(layer "F.Cu")
@@
 		)
 	)
+	(footprint ""
+		(layer "F.Cu")
+		(at 124.08 85.65)
+		(property "Reference" ""
+			(at 0 0 0)
+			(layer "F.SilkS")
+			(effects
+				(font
+					(size 1.27 1.27)
+					(thickness 0.15)
+				)
+			)
+		)
+		(property "Value" ""
+			(at 0 0 0)
+			(layer "F.Fab")
+			(effects
+				(font
+					(size 1.27 1.27)
+					(thickness 0.15)
+				)
+			)
+		)
+		(property "Footprint" ""
+			(at 0 0 0)
+			(layer "F.Fab")
+			(hide yes)
+			(effects
+				(font
+					(size 1.27 1.27)
+					(thickness 0.15)
+				)
+			)
+		)
+		(property "Datasheet" ""
+			(at 0 0 0)
+			(layer "F.Fab")
+			(hide yes)
+			(effects
+				(font
+					(size 1.27 1.27)
+					(thickness 0.15)
+				)
+			)
+		)
+		(property "Description" ""
+			(at 0 0 0)
+			(layer "F.Fab")
+			(hide yes)
+			(effects
+				(font
+					(size 1.27 1.27)
+					(thickness 0.15)
+				)
+			)
+		)
+		(pad "" smd roundrect
+			(at 0.01 0 180)
+			(size 0.9 0.95)
+			(layers "B.Cu" "B.Paste" "B.Mask")
+			(roundrect_rratio 0.25)
+			(net 1 "GND")
+			(pintype "passive")
+		)
+	)
 	(footprint "STS_connector:SAMTEC_ZF5S-08-01-T-WT"
 		(layer "B.Cu")
@@
 	)
 	(via
-		(at 135.7 85.365)
+		(at 135.68 84.27)
 		(size 0.6)
 		(drill 0.3)
@@
 	)
 	(via
-		(at 141.252 87.7)
+		(at 141.24 88.25)
 		(size 0.6)
 		(drill 0.3)
@@
 	)
 	(via
-		(at 135.7 87.725)
+		(at 135.68 86.63)
 		(size 0.6)
 		(drill 0.3)
@@
 	)
 	(via
-		(at 131.5 88.75)
+		(at 131.48 88.335)
 		(size 0.6)
 		(drill 0.3)
@@
 	)
 	(via
-		(at 131.5 89.875)
+		(at 131.48 89.46)
 		(size 0.6)
 		(drill 0.3)
@@
 	)
 	(via
-		(at 138.6 87.7)
+		(at 138.588 88.25)
 		(size 0.6)
 		(drill 0.3)
@@
 	)
 	(via
-		(at 134.5 87.725)
+		(at 134.48 86.63)
 		(size 0.6)
 		(drill 0.3)
@@
 	)
 	(via
-		(at 135.7 89.875)
+		(at 135.68 89.46)
 		(size 0.6)
 		(drill 0.3)
@@
 	)
 	(via
-		(at 133 88.75)
+		(at 132.98 88.335)
 		(size 0.6)
 		(drill 0.3)
@@
 	)
 	(via
-		(at 131.5 87.725)
+		(at 131.48 86.63)
 		(size 0.6)
 		(drill 0.3)
@@
 	)
 	(via
-		(at 134.5 85.365)
+		(at 134.48 84.27)
 		(size 0.6)
 		(drill 0.3)
@@
 	)
 	(via
-		(at 140.05 89.025)
+		(at 140.038 89.24)
 		(size 0.6)
 		(drill 0.3)
@@
 	)
 	(via
-		(at 134.5 89.875)
+		(at 134.48 89.46)
 		(size 0.6)
 		(drill 0.3)
@@
 	)
 	(via
-		(at 134.5 88.75)
+		(at 134.48 88.335)
 		(size 0.6)
 		(drill 0.3)
@@
 	)
 	(via
-		(at 133 89.875)
+		(at 132.98 89.46)
 		(size 0.6)
 		(drill 0.3)
@@
 	)
 	(via
-		(at 140.05 87.7)
+		(at 140.038 88.25)
 		(size 0.6)
 		(drill 0.3)
@@
 	)
 	(via
-		(at 135.7 86.5)
+		(at 135.68 85.405)
 		(size 0.6)
 		(drill 0.3)
@@
 	)
 	(via
-		(at 134.5 86.5)
+		(at 134.48 85.405)
 		(size 0.6)
 		(drill 0.3)
@@
 	)
 	(via
-		(at 141.252 89.025)
+		(at 141.24 89.24)
 		(size 0.6)
 		(drill 0.3)
@@
 	)
 	(via
-		(at 133 87.725)
+		(at 132.98 86.63)
 		(size 0.6)
 		(drill 0.3)
@@
 	)
 	(via
-		(at 135.7 88.75)
+		(at 135.68 88.335)
 		(size 0.6)
 		(drill 0.3)
@@
 	)
 	(via
-		(at 133 86.51)
+		(at 132.98 85.415)
 		(size 0.6)
 		(drill 0.3)
@@
 	)
 	(via
-		(at 133 85.375)
+		(at 132.98 84.28)
 		(size 0.6)
 		(drill 0.3)
@@
 	(segment
 		(start 113.3 91.07)
+		(end 114.884 89.486)
+		(width 1.5)
+		(layer "In2.Cu")
+		(net 7)
+	)
+	(segment
+		(start 113.3 91.07)
 		(end 104 91.07)
 		(width 1.5)
@@
 	)
 	(segment
+		(start 114.884 85.604)
+		(end 114.54 85.26)
+		(width 1.5)
+		(layer "In2.Cu")
+		(net 7)
+	)
+	(segment
 		(start 117.44 78.64)
 		(end 117.44 79.69)
@@
 	)
 	(segment
-		(start 114.884 86.713233)
-		(end 114.884 89.486)
-		(width 1.5)
-		(layer "In2.Cu")
-		(net 7)
-	)
-	(segment
 		(start 116.657944 75.97)
 		(end 114.54 78.087944)
@@
 	)
 	(segment
-		(start 114.54 86.369233)
-		(end 114.884 86.713233)
+		(start 114.54 85.26)
+		(end 114.54 78.087944)
 		(width 1.5)
 		(layer "In2.Cu")
@@
 	)
 	(segment
+		(start 114.884 89.486)
+		(end 114.884 85.604)
+		(width 1.5)
+		(layer "In2.Cu")
+		(net 7)
+	)
+	(segment
 		(start 126.89 82.64)
 		(end 128.04 82.64)
@@
 	)
 	(segment
-		(start 114.54 78.087944)
-		(end 114.54 86.369233)
-		(width 1.5)
-		(layer "In2.Cu")
-		(net 7)
-	)
-	(segment
-		(start 114.884 89.486)
-		(end 113.3 91.07)
-		(width 1.5)
-		(layer "In2.Cu")
-		(net 7)
-	)
-	(segment
 		(start 99.92 124.19)
 		(end 99.91 124.18)
@@
 	)
 	(via
-		(at 98.2 130.95)
+		(at 98.11 131.12)
 		(size 1)
 		(drill 0.6)
@@
 	)
 	(segment
+		(start 98.11 131.12)
+		(end 99.23 130)
+		(width 1.5)
+		(layer "In2.Cu")
+		(net 8)
+	)
+	(segment
+		(start 131.525 121.775)
+		(end 131.525 101.85)
+		(width 1.5)
+		(layer "In2.Cu")
+		(net 8)
+	)
+	(segment
 		(start 160.773 86.834887)
 		(end 158.47 89.137887)
@@
 	)
 	(segment
-		(start 98.2 130.95)
-		(end 99.15 130)
+		(start 123.3 130)
+		(end 131.525 121.775)
 		(width 1.5)
 		(layer "In2.Cu")
@@
 	)
 	(segment
-		(start 123.3 130)
-		(end 131.525 121.775)
-		(width 1.5)
-		(layer "In2.Cu")
-		(net 8)
-	)
-	(segment
 		(start 158.47 89.137887)
 		(end 158.47 94.12)
@@
 	)
 	(segment
-		(start 130.842 98.5)
-		(end 128.8 98.5)
-		(width 0.5)
+		(start 99.23 130)
+		(end 123.3 130)
+		(width 1.5)
 		(layer "In2.Cu")
 		(net 8)
 	)
 	(segment
-		(start 99.15 130)
-		(end 123.3 130)
-		(width 1.5)
+		(start 130.842 98.5)
+		(end 128.8 98.5)
+		(width 0.5)
 		(layer "In2.Cu")
 		(net 8)
@@
 	)
 	(segment
-		(start 131.525 121.775)
-		(end 131.525 101.85)
-		(width 1.5)
-		(layer "In2.Cu")
+		(start 97.87 130.88)
+		(end 97.87 128.523)
+		(width 0.3)
+		(layer "B.Cu")
 		(net 8)
 	)
@@
 	)
 	(segment
-		(start 98.2 130.95)
-		(end 97.87 130.62)
-		(width 0.3)
-		(layer "B.Cu")
-		(net 8)
-	)
-	(segment
 		(start 132.2405 98.4555)
 		(end 136.643 98.4555)
@@
 	)
 	(segment
-		(start 97.87 130.62)
-		(end 97.87 128.523)
+		(start 98.11 131.12)
+		(end 97.87 130.88)
 		(width 0.3)
 		(layer "B.Cu")
