File: Sidepanel Y/STS1_SIDEPANEL.kicad_sch (KiCad schematic)
At the start: 4 parts, among them J1 Conn_01x08

Commit message: replace ZF5S-*-01-T-WT and 2005280040 connectors with T1M-*-F-SH-L-FR connector
Parts:
- removed UV1: 501461-0491, STS_connector:200528-0040, symbol Connector:501461-0491
- added J2: Conn_01x04, STS_connector:SAMTEC_T1M-04-X-SH-L, symbol Connector_Generic:Conn_01x04
- J1: footprint STS_connector:SAMTEC_ZF5S-08-01-T-WT -> STS_connector:SAMTEC_T1M-08-F-SH-L
Connections:
- net +3V3: now also J2.01 (Pin_1)
- net GND1: now also J2.04 (Pin_4)
- net SCL: now also J2.03 (Pin_3)
- net SDA: now also J2.02 (Pin_2)
- no-connect marks 2 -> 0
